Commit message: urdf: Add Sims style diamond indicator to AMiRo models

File: catkin_ws/src/demo/urdf/amiro.urdf (robot description, URDF)
Before this commit: robot AMiRo, 4 links, 3 joints
Links:
- added link indicator; visual box size=.2 .2 .2
Joints:
- added joint base_link_to_indicator: type fixed, parent base_link, child indicator, origin xyz=0 0 1.0 rpy=0.785 0.785 0

Commit message: urdf: Add flag to AMiRo

File: catkin_ws/src/demo/urdf/amiro.urdf (robot description, URDF)
Before this commit: robot AMiRo, 5 links, 4 joints
Links:
- removed link indicator
- added link flag; visual box size=.15 .01 .1
- added link rod; visual cylinder length=1.0 radius=0.01
Joints:
- removed joint base_link_to_indicator
- added joint base_link_to_flag: type fixed, parent base_link, child flag, origin xyz=-.075 0 0.95 rpy=0 0 0
- added joint rod_link_to_base: type fixed, parent base_link, child rod, origin xyz=0 0 0.5
